File: cydonia.sch (KiCad schematic (older format))
At the start: 115 parts, among them J1 NEIGHBOR1, J19 GND, J2 NEIGHBOR2, J3 RFIN, J7 BONUS_ROW, J8 LO, U1 TLV3502, U2 AD8347, U3 SAW FILTER, U4 LNA, U5 BAND PASS FILTER, U6 ADF4360, X1 TCXO

Commit message: cydonia: initial commit, based on quince
Parts:
- removed J1: NEIGHBOR1, gsg-modules:HEADER-2x20, symbol Connector_Generic:Conn_02x20_Odd_Even
- removed J2: NEIGHBOR2, gsg-modules:HEADER-2x20, symbol Connector_Generic:Conn_02x20_Odd_Even
- removed J7: BONUS_ROW, gsg-modules:HEADER-1x20, symbol Connector_Generic:Conn_01x20
- removed MH1, MH2, MH3, MH4: MOUNTING_HOLE, gsg-modules:HOLE126MIL-COPPER, symbol Connector_Generic:Conn_01x01
- removed U1: TLV3502, gsg-modules:SOIC8-154, symbol gsg-symbols:TLV3502
- added C43: 1nF, gsg-modules:0402, symbol Device:C
- added C44: 100pF, gsg-modules:0402, symbol Device:C
- added D2, D3: LED, gsg-modules:0603D, symbol Device:LED
- added FB2: Ferrite_Bead, gsg-modules:0805, symbol Device:Ferrite_Bead
- added J1, J2: PMOD, cydonia:PinHeader_2x06_P2.54mm_PMOD, symbol Connector_Generic:Conn_02x06_Top_Bottom
- added J4: BIAS, gsg-modules:HEADER-1x2, symbol Connector_Generic:Conn_01x02
- added L8: 3.6nH, gsg-modules:0402, symbol Device:L
- added L9: 27nH, gsg-modules:0402, symbol Device:L
- added R34: 1.5k, gsg-modules:0402, symbol Device:R
- added T1: HHM1903A4, cydonia:HHM1903A4, symbol cydonia:HHM1903A4
- added U1: HHM2293A1, gsg-modules:HHM2293A1, symbol gsg-symbols:HHM2293A1
- added U7: LNA, gsg-modules:BGA7H1N6, symbol gsg-symbols:BGA5H1BN6
- C1: value 100nF -> 1nF; Description CAP CER 0.1UF 10V X5R 0402 -> CAP CER 1000PF 50V X7R 0402; Manufacturer Samsung -> Taiyo Yuden; Part Number CL05A104MP5NNNC -> UMK105B7102KV-F
- C11, C12, C13, C19, C20, C25, C27, C30, C31, C33, C35, C41: Part Number CL05A104MP5NNNC -> ‎CL05A104KP5NNNC‎
- C18: Manufacturer Samsung -> Yageo; Part Number CL05B271KB5NNNC -> CC0402KRX7R9BB271
- C28: Description CAP CER 560PF 50V X7R 0402 -> CAP CER 560PF 25V X7R 0402; Manufacturer Samsung -> Yageo; Part Number CL05B561KB5NNNC -> CC0402KRX7R8BB561
- C38: value C -> 100pF; Description (none) -> CAP CER 100PF 50V C0G/NP0 0402; Field7 (none) -> DNP; Manufacturer (none) -> Samsung; Note DNP -> (none); Part Number (none) -> CL05C101JB5NNNC
- D1: Description TVS DIODE 4V 1005 -> 5.5V, ESD PROTECTION DEVICES, DF; Manufacturer Murata -> Micro Commercial Components; Part Number LXES15AAA1-153 -> ESDSLC5V0L2B-TP
- R17: value 0 -> 1.5k; Description RES SMD 0 OHM JUMPER 1/16W 0402 -> RES SMD 1.5K OHM 5% 1/16W 0402; Note DNP -> (none); Part Number RC0402JR-070RL -> RC0402JR-071K5L
- R2: value 0 -> 100; Description RES SMD 0 OHM JUMPER 1/16W 0402 -> RES SMD 100 OHM 5% 1/16W 0402; Part Number RC0402JR-070RL -> RC0402JR-07100RL
Connections:
- net labels added: CLK, DATA, EN, I_N, I_P, LE, Q_N, Q_P, RF_N, RF_P
- net labels removed: +5V, ADC0_0, ADC0_2, ADC0_5, CLK0, CLK2, I2C0_SCL, I2C0_SDA, IN_A+, IN_A-, IN_B+, IN_B-, OUT_A, OUT_B, P0_0, P0_1, P1_0, P1_1, P1_10, P1_11, P1_12, P1_13, P1_14, P1_15, P1_16, P1_17, P1_18, P1_19, P1_2, P1_20, P1_3, P1_4, P1_5, P1_6, P1_7, P1_8, P1_9, P2_0, P2_1, P2_10, P2_11, P2_12, P2_13, P2_2, P2_3, P2_4, P2_5, P2_6, P2_7, P2_8, P2_9, P3_0, P3_1, P3_2, P3_3, P3_4, P3_5, P3_6, P3_7, P4_0, P4_10, P4_2, P4_3, P4_4, P4_5, P4_6, P4_7, P4_8, P4_9, P5_0, P5_1, P5_2, P5_3, P5_4, P5_5, P5_6, P5_7, P6_0, P6_1, P6_10, P6_2, P6_3, P6_4, P6_5, P6_6, P6_7, P6_8, P6_9, P7_0, P7_1, P7_2, P7_7, P9_5, P9_6, PF_4, RESET, RTC_ALARM, VBAT, VCC, WAKEUP0
- wire segments 468 -> 435
- no-connect marks 86 -> 5
Other:
- note added: "I channel inverted"
- note removed: "BOOT"
- note removed: "CIPO"
- note removed: "COPI"
- note removed: "CS"
- note removed: "DFU"
- note removed: "ISP"
- note removed: "Interpret SGPIO0 as Q\nand SGPIO1 as I."
- note removed: "SCK"
- note removed: "SGPIO0"
- note removed: "SGPIO1"
- note removed: "TODO\nI2C I/O expander\nmaybe 3.3 V voltage regulator\nmaybe replace U6 with CC2500"
- note removed: "VGIN DAC/ADC option"
- note removed: "both channels inverted"
- note removed: "option to use LPC4330\nCLKOUT as reference clock"
- moved on the sheet: C2, C7, C9, D1, FB1, J19, J3, L4, R12, R3, R4, R5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
